File: hardware/PGTN021_octasource_controls.brd (EAGLE design)
At the start: 69.8 x 100.3 mm, 87 parts

Commit message: Changed resistor values to 39k
Parts:
- R1, R2, R3, R4, R5, R6: value 75k -> 39k
