File: hardware/PGTN021_octasource_led_drivers.brd (EAGLE design)
At the start: 69.8 x 100.3 mm, 138 parts, among them IC1 TL084P, IC2 TL084P, IC3 TL084P, IC4 TL084P

Commit message: added capacitor values
Parts:
- C1, C2, C3, C4, C5, C6, C7, C8: value (none) -> 100nF
