File: hardware/mkiii/PGTN021_octasource_mkiii_panel.sch (EAGLE design)
At the start: 20 parts

Commit message: Final mkiii hardware
Parts:
- added H21: MOUNT-PAD-ROUND6.5, holes:MOUNT-PAD-ROUND6.5
Connections:
- removed net N$5: H11.MOUNT, H15.MOUNT
- removed net N$7: H12.MOUNT, H16.MOUNT
- removed net N$8: H13.MOUNT, H17.MOUNT
- new net N$3: H19.MOUNT
- net N$1: now also H10.MOUNT, H11.MOUNT, H12.MOUNT, H13.MOUNT, H14.MOUNT, H15.MOUNT, H16.MOUNT, H17.MOUNT, H21.MOUNT, H9.MOUNT
- net N$4: now also H20.MOUNT; no longer H10.MOUNT, H14.MOUNT
Other:
- moved on the sheet: H9
