File: hardware/mkiii/PGTN021_octasource_mkiii_controls.brd (EAGLE design)
At the start: 69.9 x 110.5 mm, 139 parts, among them IC1 IS32FL3738, SW1 ENCODER_SW1-PEC12, U1 74AHCT1G125"

Commit message: Final mkiii hardware
Parts:
- removed IO11, IO12, IO13, IO14, IO15: HEADER/MALE/01, connectors:HEADER/MALE/01
- added 3.3VA: HEADER/MALE/01, connectors:HEADER/MALE/01
- added AUX: WQP-PJ301M-12_JACK, controls:WQP-PJ301M-12_JACK
- added R1_A, R2_A, R3_A, R4_A, R5_B, R6_A, R7_A, R8_B: 0R, resistors:R0603
- moved PT2 10.2 mm to (68.6, 66.0)
- moved PT4 10.2 mm to (68.6, 71.1)
- moved PT6 10.2 mm to (68.6, 55.9)
- moved PT8 10.2 mm to (68.6, 61.0)
- moved PT1 10.2 mm to (68.6, 63.5)
- moved PT3 10.2 mm to (68.6, 68.6)
- moved PT5 10.2 mm to (68.6, 53.3)
- moved PT7 10.2 mm to (68.6, 58.4)
- moved VR3 2.29 mm to (11.4, 72.4)
- moved LED1 1.91 mm to (36.8, 34.8)
- moved LED2 1.91 mm to (43.0, 32.1)
- moved LED3 1.91 mm to (30.8, 32.2)
- moved LED4 1.91 mm to (45.6, 26.0)
- moved LED6 1.91 mm to (30.7, 19.9)
- moved LED7 1.91 mm to (43.0, 19.8)
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Connections:
- new net -5V: -5V.1, R6_A.2, S1.4
- new net 3.3VA: 3.3VA.1, R5_B.2
- new net N$14: AUX.P$1, CV6.1
- new net N$15: CV4_.1, R1_A.1
- new net N$17: CV3_.1, R2_A.1
- new net N$18: CV2_.1, R3_A.1
- new net N$19: CV5_.1, R4_A.1
- new net N$21: R5_B.1, R6_A.1, VR1.1, VR2.1, VR3.1, VR4.1
- net +5V: now also R7_A.2
- net 3.3V: no longer VR1.1, VR2.1, VR3.1, VR4.1
- net N$10: now also R4_A.2
- net N$11: now also R7_A.1, R8_B.1, VR1.3, VR2.3, VR3.3, VR4.3; no longer -5V.1, S1.4
- net N$2: now also R1_A.2
- net N$7: now also R2_A.2
- net N$9: now also R3_A.2
- net PE: now also AUX.P$2, AUX.P$3, R8_B.2; no longer VR1.3, VR2.3, VR3.3, VR4.3
Routing:
- net N$14: track 0.00 -> 110.4 mm
- net N$21: track 0.00 -> 84.0 mm, vias 0 -> 1
- net -5V: track 0.00 -> 79.2 mm, vias 0 -> 1
- net 3.3V: track 184.4 -> 106.7 mm, vias 1 -> 0
- net N$9: track 66.6 -> 112.9 mm, vias 0 -> 1
- net N$7: track 48.3 -> 86.8 mm
- net N$2: track 31.7 -> 61.9 mm, vias 0 -> 1
- net N$10: track 55.4 -> 83.7 mm, vias 0 -> 1
- net 3.3VA: track 0.00 -> 20.2 mm, vias 0 -> 1
- net N$50: track 135.1 -> 122.8 mm
- net N$11: track 65.6 -> 76.5 mm
- net PE: track 51.9 -> 42.6 mm, vias 5 -> 6
- net N$66: track 175.5 -> 168.3 mm
- net +5V: track 23.3 -> 29.0 mm, vias 1 -> 2
- net N$51: track 134.9 -> 129.3 mm
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Other:
- board text added: "OCTOSOURCE"
- board text removed: "OCTASOURCE"

Commit message: add photo of mkii
Parts:
- U1: value 74AHCT1G125" -> 74AHCT1G125
Other:
- board text added: "74AHCT1G125"
