File: hardware/mkiii/PGTN021_octasource_mkiii_controls.sch (EAGLE design)
At the start: 138 parts, among them IC1 IS32FL3738, SW1 ENCODER_SW1-PEC12, U1 74AHCT1G125"

Commit message: Final mkiii hardware
Parts:
- removed IO11, IO12, IO13, IO14, IO15: HEADER/MALE/01, connectors:HEADER/MALE/01
- added 3.3VA: HEADER/MALE/01, connectors:HEADER/MALE/01
- added AUX: WQP-PJ301M-12_JACK, controls:WQP-PJ301M-12_JACK
- added R1_A, R2_A, R3_A, R4_A, R5_B, R6_A, R7_A, R8_B: 0R, resistors:RESISTOR
Connections:
- new net -5V: -5V.3, R6_A.2, S1.4
- new net 3.3VA: 3.3VA.3, R5_B.2
- new net N$14: AUX.2, CV6.3
- new net N$15: CV4_.3, R1_A.1
- new net N$17: CV3_.3, R2_A.1
- new net N$18: CV2_.3, R3_A.1
- new net N$19: CV5_.3, R4_A.1
- new net N$21: R5_B.1, R6_A.1, VR1.A, VR2.A, VR3.A, VR4.A
- net +5V: now also R7_A.2
- net 3.3V: no longer VR1.A, VR2.A, VR3.A, VR4.A
- net N$10: now also R4_A.2
- net N$11: now also R7_A.1, R8_B.1, VR1.E, VR2.E, VR3.E, VR4.E; no longer -5V.3, S1.4
- net N$2: now also R1_A.2
- net N$7: now also R2_A.2
- net N$9: now also R3_A.2
- net PE: now also AUX.1, AUX.3, R8_B.2; no longer VR1.E, VR2.E, VR3.E, VR4.E
Other:
- note added: "Populate either A or B resistors"
- moved on the sheet: -5V, 5, 5V, CV2_, CV3_, CV4_, CV5_, CV6, PT1, PT2, PT3, PT4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

Commit message: add photo of mkii
Parts:
- U1: value 74AHCT1G125" -> 74AHCT1G125
Changed lines of the file:
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@@
 <attribute name="SPICEPREFIX" value="G"/>
 </part>
-<part name="U1" library="ic_digital" deviceset="74AHCT1G125" device="&quot;"/>
+<part name="U1" library="ic_digital" deviceset="74AHCT1G125" device="&quot;" value="74AHCT1G125"/>
 <part name="SUPPLY27" library="supply" deviceset="GND" device="">
 <attribute name="SPICEPREFIX" value="G"/>
