File: hardware/mkiii/PGTN021_octasource_mkiii_panel.brd (EAGLE design)
At the start: 70.5 x 128.6 mm, 25 parts

Commit message: Final mkiii hardware
Parts:
- added H21: MOUNT-PAD-ROUND6.5, holes:6.5-PAD
- moved U$2 3.18 mm to (37.5, -1.91)
- moved H14 2.29 mm to (11.4, 72.4)
- moved H1 1.91 mm to (36.8, 43.8)
- moved H16 1.91 mm to (58.4, 73.7)
- moved H19 1.91 mm to (62.9, 6.35)
- moved H2 1.91 mm to (49.5, 38.7)
- moved H3 1.91 mm to (54.6, 26.0)
- moved H4 1.91 mm to (49.5, 13.3)
- moved H5 1.91 mm to (36.8, 8.26)
- moved H7 1.91 mm to (19.1, 26.0)
- moved H9 1.91 mm to (13.3, 48.3)
- moved H20 1.90 mm to (10.8, 6.35)
- moved H6 1.90 mm to (24.1, 13.3)
- moved H8 1.90 mm to (24.1, 38.7)
- moved H10 1.80 mm to (22.9, 55.2)
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Connections:
- removed net N$5: H11.B6.5, H15.B7.5
- removed net N$7: H12.B6.5, H16.B7.5
- removed net N$8: H13.B6.5, H17.B7.5
- new net N$3: H19.B6.5
- net N$1: now also H10.B6.5, H11.B6.5, H12.B6.5, H13.B6.5, H14.B7.5, H15.B7.5, H16.B7.5, H17.B7.5, H21.B6.5, H9.B6.5
- net N$4: now also H20.B5; no longer H10.B6.5, H14.B7.5
Routing:
- net N$1: track 61.2 -> 288.1 mm
- net N$2: track 118.4 -> 1.74 mm
- net N$8: track 55.8 -> 0.00 mm
- net N$7: track 21.6 -> 0.00 mm
- net N$4: track 21.6 -> 0.00 mm
- net N$5: track 20.3 -> 0.00 mm
Other:
- board text added: "JLCJLCJLCJLC"
